File: hardware/kicad/meshtastic-node.kicad_sch (KiCad schematic)
At the start: 18 parts, among them Q1 AO3401A, SW1 rocker ON/OFF, SW2 user button, U1 ESP32-S3-DevKitC-1, U2 E22-400M22S (SX1268), U3 GY-NEO8MV2, U4 SSD1306 128x64, U5 TP4056, U6 TPS63020

Commit message: Move LORA_DIO1 to GPIO17 and leave RXEN unconnected
The E22-400M22S's DIO1 is soldered to GPIO17, not GPIO15, and DIO2_AS_RF_SWITCH
covers RX/TX switching without a dedicated RXEN GPIO. Updates the harness,
netlist, and KiCad schematic to match.

Co-Authored-By: Claude Sonnet 5 <noreply@anthropic.com>
Connections:
- net LORA_DIO1: now also U1.GPIO17; no longer U1.GPIO15
- net LORA_RXEN: no longer names the net of U2.RXEN
- net LORA_RXEN: no longer U1.GPIO17
Changed lines of the file:
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@@
     (effects (font (size 1.27 1.27)) (justify left))
   )
-  (label "LORA_DIO1" (at 110.32 130.16 180)
+  (label "LORA_DIO1" (at 110.32 135.24 180)
     (effects (font (size 1.27 1.27)) (justify left))
   )
@@
   )
   (label "LORA_NRST" (at 220.32 111.35 180)
-    (effects (font (size 1.27 1.27)) (justify left))
-  )
-  (label "LORA_RXEN" (at 110.32 135.24 180)
-    (effects (font (size 1.27 1.27)) (justify left))
-  )
-  (label "LORA_RXEN" (at 220.32 113.89 180)
     (effects (font (size 1.27 1.27)) (justify left))
   )
@@
   )
   (symbol_instances
-    (path "/c709f035-7dde-4bfb-9a0a-a2c2d14464c8"
+    (path "/83ac34c7-1bed-4e47-9514-4911cf44583c"
       (reference "U1") (unit 1) (value "ESP32-S3-DevKitC-1") (footprint "")
     )
-    (path "/d475e183-04fd-4d10-837c-3d54e80d5a4d"
+    (path "/8a7e6946-294c-4c88-8aab-15a730813a29"
       (reference "U2") (unit 1) (value "E22-400M22S (SX1268)") (footprint "")
     )
-    (path "/57d6e93b-f92d-4903-b625-d8d779e80037"
+    (path "/1e0c5de2-7faf-46c3-83c2-78d0acc0fc2d"
       (reference "U3") (unit 1) (value "GY-NEO8MV2") (footprint "")
     )
-    (path "/cced5920-86af-41a3-9869-0f71a6b8a098"
+    (path "/b547bfdb-53d0-4a81-8e51-3f389cc51d35"
       (reference "U4") (unit 1) (value "SSD1306 128x64") (footprint "")
     )
-    (path "/2484cda1-9ba2-44f1-bd37-93abc4b7908d"
+    (path "/eff0fdc4-eafb-4440-86d1-c99e18edb10e"
       (reference "U5") (unit 1) (value "TP4056") (footprint "")
     )
-    (path "/4d82a1e3-5c05-452c-b2a1-5e35ad64da7d"
+    (path "/d5543011-801d-451c-8e8b-d382cbfad42f"
       (reference "U6") (unit 1) (value "TPS63020") (footprint "")
     )
-    (path "/8e8c1d12-9d7e-44cf-86b8-4542ca0408a3"
+    (path "/ab36b4fd-c08a-4b38-8fc7-ff556d42990b"
       (reference "Q1") (unit 1) (value "AO3401A") (footprint "")
     )
-    (path "/f27627bf-67d1-4d43-94d1-16e5aff71d51"
+    (path "/2035d82a-f7db-41e2-9da0-47f1f9ef73cd"
       (reference "R1") (unit 1) (value "100k 1%") (footprint "")
     )
-    (path "/655d7195-0834-40fb-81d1-e11abde1153c"
+    (path "/361efd1b-9871-4ab1-b32d-852fdf8edfab"
       (reference "R2") (unit 1) (value "100k 1%") (footprint "")
     )
-    (path "/891c2111-4854-4eb4-825c-7f4da77f8e20"
+    (path "/ebddf768-013a-4df9-b7e9-bd8a179b49f6"
       (reference "R3") (unit 1) (value "100k") (footprint "")
     )
-    (path "/fc86f714-9203-4987-b46e-95e6bd56bf97"
+    (path "/a25eee61-3be5-49ee-86af-86ceaa15ba76"
       (reference "C1") (unit 1) (value "470u 10V low-ESR") (footprint "")
     )
-    (path "/da548dce-149c-4981-819f-38b2d27070b8"
+    (path "/a9d45a91-edc4-4c49-8964-e2048e882a72"
       (reference "C2") (unit 1) (value "10u 25V X7R") (footprint "")
     )
-    (path "/628cc0f2-6fd7-4fd5-86b6-ea05beb98ebc"
+    (path "/b3d039cc-9aa5-4728-87d0-f7e27af3630a"
       (reference "C3") (unit 1) (value "100n 50V X7R") (footprint "")
     )
-    (path "/60b27d8a-8adb-46dc-9779-b36bb1018e90"
+    (path "/377813e0-58fe-46a2-93a6-f8002e12b7c6"
       (reference "C4") (unit 1) (value "100n 50V X7R") (footprint "")
     )
-    (path "/7135a9ce-7596-4b1e-bc9b-9203b17fb399"
+    (path "/44a3b9e2-7096-42a3-bed3-d369d66373cf"
       (reference "SW1") (unit 1) (value "rocker ON/OFF") (footprint "")
     )
-    (path "/48c7565f-e58f-4e02-9580-8ae01a7ebf74"
+    (path "/0ea1dbd5-f87c-4ee9-a280-6ee1db4cc81d"
       (reference "SW2") (unit 1) (value "user button") (footprint "")
     )
-    (path "/d5b532bc-a2f4-4bf3-92d6-1ca536217fc0"
+    (path "/ccd13bf1-dae8-4c8f-9d43-963fe50d209c"
       (reference "BT1") (unit 1) (value "18650 protected") (footprint "")
     )
-    (path "/2c684270-915b-4069-bf4b-57f017c47b68"
+    (path "/38902201-001a-4f21-8ba9-5ce474f51689"
       (reference "BT2") (unit 1) (value "18650 protected") (footprint "")
     )
